File: remoteLab.kicad_sch (KiCad schematic)
At the start: 0 parts

Commit message: session 1
Parts:
- added C1: 100nF, symbol Device:C
- added D1: Status LED, symbol Device:LED
- added F1: Polyfuse, symbol Device:Polyfuse
- added J1: RPi_40pi_Hat, symbol Connector:Raspberry_Pi_4
- added J2: Debug UART, symbol Connector:Conn_01x03_Pin
- added J3: HAT_Power_Supply, symbol Connector:USB_C_Receptacle_PowerOnly_6P
- added J4: RPi powerback, symbol Connector:Conn_01x03_Pin
- added JP1, JP2, JP3: ~, symbol Jumper:SolderJumper_3_Bridged12
- added R1: 10k, symbol Device:R
- added R2, R3: 0, symbol Device:R
- added R4, R5: 10K, symbol Device:R
- added R6: 330, symbol Device:R
- added R7, R8: 5.1K, symbol Device:R
- added SW1: SW_SPDT_MSM, Button_Switch_THT:SW_CK_JS202011AQN_DPDT_Angled, symbol Switch:SW_SPDT_MSM
- added TP1, TP2, TP3, TP4: ~, symbol Connector:TestPoint
- added U1: MCP23017_SO, Package_SO:SOIC-28W_7.5x17.9mm_P1.27mm, symbol Interface_Expansion:MCP23017_SO
- added U2: ULN2803A, symbol Transistor_Array:ULN2803A
Connections:
- new net: R2.2, TP1.1, U1.13 (SDA)
- new net: R3.1, TP2.1, U1.12 (SCK)
- new net: JP2.2 (C), U1.16 (A1)
- new net: J1.10 (GPIO15/UART_RXD), J2.2 (Pin_2)
- new net: J1.14 (GND), J1.20 (GND), J1.25 (GND), J1.30 (GND), J1.34 (GND), J1.39 (GND), J1.6 (GND), J1.9 (GND)
- new net: J1.32 (GPIO12/PWM0), R6.2
- new net: J1.8 (GPIO14/UART_TXD), J2.1 (Pin_1)
- new net: D1.2 (A), R6.1
- new net: R1.2, U1.18 (~{RESET})
- new net: J3.A5 (CC1), R7.1
- new net: J3.B5 (CC2), R8.2
- new net: JP3.2 (C), U1.15 (A0)
- new net: JP1.2 (C), U1.17 (A2)
- new net +3V3: C1.1, J1.1 (3V3), J1.17 (3V3), JP1.3 (B), JP2.3 (B), JP3.3 (B), R1.1, R4.2, R5.1, U1.9 (VDD)
- new net +5V: SW1.2 (3), U2.10 (COM)
- new net +5V_EXT: F1.2, J3.A9 (VBUS), J3.B9 (VBUS), J4.3 (Pin_3), SW1.1
- new net +5V_RPI: F1.1, J1.2 (5V), J1.4 (5V), J4.2 (Pin_2), SW1.3 (4)
- new net GND: C1.2, D1.1 (K), J2.3 (Pin_3), J3.A12 (GND), J3.B12 (GND), J3.S1 (SHIELD), JP1.1 (A), JP2.1 (A), JP3.1 (A), R7.2, R8.1, U1.10 (VSS), U2.9 (GND)
- new net PWR_RELAY_0: U1.21 (GPA0), U2.1 (I1)
- new net PWR_RELAY_1: U1.22 (GPA1), U2.2 (I2)
- new net PWR_RELAY_2: U1.23 (GPA2), U2.3 (I3)
- new net RPI_PIN15: J1.15 (GPIO22/SDIO_CLK), TP3.1, U1.19 (INTB)
- new net RPI_PIN16: J1.16 (GPIO23/SDIO_CMD), TP4.1, U1.20 (INTA)
- new net RPI_SCL: J1.5 (SCL_I2C1/GPIO03), R3.2, R4.1
- new net RPI_SDA: J1.3 (SDA_I2C1/GPIO02), R2.1, R5.2
- new net SIGNAL_RELAY_0: U1.24 (GPA3)
- new net SIGNAL_RELAY_1: U1.25 (GPA4)
- new net SIGNAL_RELAY_2: U1.26 (GPA5)
- new net USB_SWITCH_0: U1.1 (GPB0)
- new net USB_SWITCH_1: U1.2 (GPB1)
- new net USB_SWITCH_2: U1.3 (GPB2)
- no-connect marks 0 -> 1
Other:
- note added: "3A polyfuse for double power supply protection"
- note added: "A0: GND A1: GND A2: GND 0b0100_A2A1A0 = 0b0100_000 Default Address: 0X20 (8bit)"
- note added: "DNP"
- note added: "R4 an R5 can be placed when stacking up multiple boards"
- note added: "SW1 allows powering the 5V net either from RPi or externally"

Commit message: session 2
Parts:
- removed U2: ULN2803A, symbol Transistor_Array:ULN2803A
- added J5: Inter-board connector, symbol Connector:Conn_01x08_Pin
Connections:
- net +3V3: now also J5.8 (Pin_8)
- net +5V: now also J5.7 (Pin_7)
- net GND: now also J2.1 (Pin_1), J5.1 (Pin_1); no longer J2.3 (Pin_3)
- net RPI_SCL: now also J5.2 (Pin_2)
- net RPI_SDA: now also J5.3 (Pin_3)
- net RPI_UART_RX: now reaches J1.10 (GPIO15/UART_RXD), J2.2 (Pin_2)
- net RPI_UART_TX: now reaches J1.8 (GPIO14/UART_TXD)
- net RPI_UART_TX: now also J2.3 (Pin_3); no longer J2.1 (Pin_1)
- net PWR_RELAY_0 renamed PWR_RELAY_CMD_0
- net PWR_RELAY_1 renamed PWR_RELAY_CMD_1
- net PWR_RELAY_2 renamed PWR_RELAY_CMD_2
- net SIGNAL_RELAY_0 renamed SIGNAL_RELAY_CMD_0
- net SIGNAL_RELAY_1 renamed SIGNAL_RELAY_CMD_1
- net SIGNAL_RELAY_2 renamed SIGNAL_RELAY_CMD_2
- net USB_SWITCH_0 renamed USB_SWITCH_CMD_0
- net USB_SWITCH_1 renamed USB_SWITCH_CMD_1
- net USB_SWITCH_2 renamed USB_SWITCH_CMD_2
Other:
- added sheet relay (relay.kicad_sch)
- moved on the sheet: C1, D1, F1, J1, J2, J3, J4, JP1, JP2, JP3, R1, R2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

Commit message: session 3
Parts:
- removed F1: Polyfuse, symbol Device:Polyfuse
- removed J4: RPi powerback, symbol Connector:Conn_01x03_Pin
- removed SW1: SW_SPDT_MSM, Button_Switch_THT:SW_CK_JS202011AQN_DPDT_Angled, symbol Switch:SW_SPDT_MSM
- added C3: 100uF, symbol Device:C
- added D3: LED, symbol Device:LED
- added Q1, Q2: AO4407, Package_SO:SOIC-8_3.9x4.9mm_P1.27mm, symbol Transistor_FET:IRF7404
- added R10: 100k, symbol Device:R
- added R13: 330, symbol Device:R
- added U4: LTC4412xS6, Package_TO_SOT_SMD:TSOT-23-6, symbol Power_Management:LTC4412xS6
Connections:
- net +5V_RPI is gone; now on net +5V: J1.2 (5V), J1.4 (5V)
- net +5V: now also C3.1, D3.2 (A), Q1.5 (D), Q1.6 (D), Q1.7 (D), Q1.8 (D), R10.2, U4.6 (SENSE)
- net +5V_EXT: now also Q2.5 (D), Q2.6 (D), Q2.7 (D), Q2.8 (D), U4.1 (VIN)
- net GND: now also C3.2, U4.2 (GND), U4.3 (CTL)
- new net: R13.1, U4.4 (STAT)
- new net: D3.1 (K), R13.2
- new net: Q1.1 (S), Q1.2 (S), Q1.3 (S), Q2.1 (S), Q2.2 (S), Q2.3 (S)
- new net: Q1.4 (G), Q2.4 (G), R10.1, U4.5 (GATE)
- no-connect marks 1 -> 0
Other:
- note removed: "3A polyfuse for double power supply protection"
- note removed: "SW1 allows powering the 5V net either from RPi or externally"
- moved on the sheet: D1, J3, R6, R7, R8

Commit message: session 4
Parts:
- removed R10: 100k, symbol Device:R
- added C2: 10uF, symbol Device:C
Connections:
- net +5V: now also Q1.1 (S), Q1.2 (S), Q1.3 (S), R13.2; no longer D3.2 (A), Q1.5 (D), Q1.6 (D), Q1.7 (D), Q1.8 (D)
- net +5V_EXT: now also Q2.1 (S), Q2.2 (S), Q2.3 (S), C2.1; no longer Q2.5 (D), Q2.6 (D), Q2.7 (D), Q2.8 (D)
- net GND: now also C2.2
- net at R13.1: now also D3.2 (A); no longer U4.4 (STAT)
- net at D3.1 (K): now also U4.4 (STAT); no longer R13.2
- new net: Q1.5 (D), Q1.6 (D), Q1.7 (D), Q1.8 (D), Q2.5 (D), Q2.6 (D), Q2.7 (D), Q2.8 (D)
Other:
- moved on the sheet: D3, Q2, R13

Commit message: session 5
Parts:
- removed Q1, Q2: AO4407, Package_SO:SOIC-8_3.9x4.9mm_P1.27mm, symbol Transistor_FET:IRF7404
- added D2: SMAJ5.0A, Diode_SMD:D_SMA, symbol Diode:SMAJ5.0A
- added Q3: IRF7324, Package_SO:SOIC-8_3.9x4.9mm_P1.27mm, symbol Transistor_FET:IRF7324
Connections:
- net +5V: now also Q3.3 (S2)
- net +5V_EXT: now also D2.1 (A1), Q3.1 (S1)
- net GND: now also J1.14 (GND), J1.20 (GND), J1.25 (GND), J1.30 (GND), J1.34 (GND), J1.39 (GND), J1.6 (GND), J1.9 (GND), D2.2 (A2)
- net RPI_PIN18: now reaches J1.18 (GPIO24/SDIO_DAT0)
- net RPI_MOSI: now reaches J1.19 (MOSI_SPI0/GPIO10)
- net RPI_MISO: now reaches J1.21 (MISO_SPI0/GPIO09)
- net RPI_PIN22: now reaches J1.22 (GPIO25/SDIO_DAT1)
- net RPI_SCLK: now reaches J1.23 (SCLK_SPI0/GPIO11)
- net RPI_CE0: now reaches J1.24 (~{CE0}_SPI0/GPIO08)
- net at U4.5 (GATE): now also Q3.2 (G1), Q3.4 (G2)
- net RPI_UART_RX: no longer names the net of J1.10 (GPIO15/UART_RXD), J2.2 (Pin_2)
- net RPI_UART_TX: no longer names the net of J1.8 (GPIO14/UART_TXD), J2.3 (Pin_3)
- new net: Q3.5 (D2), Q3.6 (D2), Q3.7 (D1), Q3.8 (D1)
Other:
- added sheet uart+usb (uart+usb.kicad_sch)
- note added: "5V_RPI and 5V belong to the same net so that one power source can e used to power both the RPi and the Hat"
- note added: "D2 is a TVS diode to protect aginst ESD"
- note added: "This is a power source Or-ing design. The LTC4412 with B-to-B P-MOSFETs act as an ideal diode to isolate the two power sources: 5V_EXT and 5V_RPI and protect them from fighting eachother when boath are plugged in."
- moved on the sheet: C1, C2, C3, D1, D3, J1, J2, J3, J5, JP1, JP2, JP3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
